Commit message: fairino_description: ajouter le repere flange sur FR10 et FR20
L'URDF s'arretait a wrist3_link, dont l'origine est a l'interieur du
poignet et non sur la face de montage de l'effecteur. Tout outil greffe
sur wrist3_link etait donc decale de l'epaisseur de bride, sans que rien
ne le signale.

Ajout d'un link flange, enfant fixe de wrist3_link, purement translate
sur son axe Z sans rotation :
  - FR10 : 0.106 m
  - FR20 : 0.120 m

Cotes relevees sur les plans constructeur, ajoutes dans doc/ et installes
dans le share/ du paquet : le FR10 porte 114 | 106 et le FR20 138 | 120,
ou les 114 et 138 correspondent aux origines de j6 deja presentes dans
les URDF, ce qui confirme les offsets de bride.

Les moveit2_config incluent ces URDF par xacro, le flange s'y propage
sans duplication. Les SRDF gardent tip_link=wrist3_link et sont
inchanges.

File: fairino_description/urdf/fairino10_v6.urdf (robot description, URDF)
Before this commit: robot fairino10_v6_robot, 7 links, 6 joints
Links:
- added link flange
Joints:
- added joint wrist3_to_flange: type fixed, parent wrist3_link, child flange, origin xyz=0 0 0.106 rpy=0 0 0

File: fairino_description/urdf/fairino20_v6.urdf (robot description, URDF)
Before this commit: robot fairino20_v6_robot, 7 links, 6 joints
Links:
- added link flange
Joints:
- added joint wrist3_to_flange: type fixed, parent wrist3_link, child flange, origin xyz=0 0 0.120 rpy=0 0 0
